File: Electrical/Titan_R3/Titan_R3.kicad_pcb (KiCad board)
At the start: 4 copper layers, 40 x 80 mm, 99 parts, among them IC1 NEO-M9N-00B, J1 BATT, J10 UART, J11 SPI, J12 PROPY, J13 PROPZ, J14 TVCY, J15 GPS ANT, J16 TVCZ, J17 PYRO 1, J18 PYRO 2, J19 PYRO 3, J2 12V OUT, J20 PYRO 4, J21 DM3D-SF, J3 USB_C_Receptacle_USB2.0, J4 5V OUT, J5 SW, J6 3V3 OUT, J7 PYRO ARM, J8 SWD, J9 I2C, Q1 PYRO 1, Q2 PYRO 2, Q3 PYRO 3, Q4 PYRO 4, U1 AP63300WU-7, U2 AZ1117-3.3, U3 USBLC6-2P6, U4 ATSAMD51J19A-A, U5 BMP280, U6 SST26VF032B-104I_SM, U7 BMI088, U8 LSM9DS1TR, Y1 32.768

Commit message: worked more on routing
Parts:
- moved C14 4.16 mm to (45.3, 52.2), turned to 0 degrees
- moved C15 2.30 mm to (48.0, 57.9)
- moved C19 1.90 mm to (45.1, 55.5)
- moved C16 1.90 mm to (45.1, 54.0)
- moved C18 1.87 mm to (39.6, 53.1), turned to 90 degrees
- moved L2 1.67 mm to (42.7, 53.0), turned to -90 degrees
- moved C13 0.30 mm to (36.7, 69.3)
- moved C8 0.13 mm to (42.4, 57.7)
- moved R9 0.13 mm to (42.4, 59.2)
- moved C11 0.10 mm to (47.8, 64.8)
Routing:
- net VCC: track 23.2 -> 94.7 mm, vias 0 -> 2
- net RESET: track 40.3 -> 64.7 mm, vias 3 -> 4
- net +5V: track 44.6 -> 64.8 mm, vias 2 -> 3
- net X_1: track 0.00 -> 8.10 mm, vias 0 -> 1
- net X_2: track 0.00 -> 5.45 mm, vias 0 -> 1
- net GND: track 20.5 -> 25.2 mm, vias 28 -> 30
- net /VDDCORE_C: track 5.39 -> 1.52 mm
- net Net-(L2-Pad2): track 2.24 -> 3.81 mm
- net +3V3: track 15.2 -> 15.1 mm, vias 9 -> 10

Commit message: major flight software changes
Parts:
- removed C25: 0.22uF, Capacitor_SMD:C_0603_1608Metric
- removed C27: 100nF, Capacitor_SMD:C_0603_1608Metric
- removed U8: LSM9DS1TR, digikey-footprints:LGA-24_3x3.5mm_LSM9DS1
- moved R14 13.6 mm to (34.7, 52.6)
- moved R16 13.6 mm to (34.7, 51.1)
- moved J6 3.51 mm to (51.0, 23.2), turned to 180 degrees
- moved J4 3.32 mm to (30.5, 23.2), turned to 180 degrees
- moved J11 3.25 mm to (21.6, 66.6)
- moved C11 2.99 mm to (46.1, 67.3), turned to -90 degrees
- moved TP1 2.45 mm to (47.3, 30.7)
- moved C15 1.64 mm to (46.6, 56.9)
- moved C18 0.98 mm to (38.9, 53.7), turned to 180 degrees
- moved R13 0.84 mm to (26.1, 72.5)
- moved Q1 0.79 mm to (26.1, 75.1)
- moved J15 0.56 mm to (39.1, 23.6)
- moved C26 0.25 mm to (28.6, 46.0)
- moved C22 0.15 mm to (39.7, 29.1)
- moved L3 0.15 mm to (33.6, 29.1)
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Connections:
- C23 pad 1: Net-(C23-Pad1) -> +3V3
- C24 pad 1: Net-(C24-Pad1) -> +3V3
- U4 pad 27: unconnected-(U4-Pad27) -> PY_3
- U4 pad 28: unconnected-(U4-Pad28) -> PY_4
- U4 pad 35: unconnected-(U4-Pad35) -> PY_1
- U4 pad 36: unconnected-(U4-Pad36) -> PY_2
- U7 pad 11: Net-(C23-Pad1) -> +3V3
- U7 pad 3: Net-(C24-Pad1) -> +3V3
Routing:
- net +12V: track 23.8 -> 88.1 mm
- net GND: track 25.2 -> 88.4 mm, vias 30 -> 106
- net R_OUT: track 0.00 -> 61.9 mm
- net +5V: track 64.8 -> 126.1 mm, vias 3 -> 4
- net SD_CS: track 0.00 -> 56.7 mm, vias 0 -> 3
- net MOSI: track 0.00 -> 55.2 mm, vias 0 -> 3
- net MISO: track 0.00 -> 52.2 mm, vias 0 -> 4
- net SCK: track 0.00 -> 50.2 mm, vias 0 -> 5
- net SCL1: track 0.00 -> 42.0 mm, vias 0 -> 2
- net SDA1: track 0.00 -> 40.2 mm, vias 0 -> 4
- net TVCY: track 0.00 -> 36.2 mm, vias 0 -> 1
- net PROPY: track 0.00 -> 35.5 mm, vias 0 -> 1
- net PY_3: track 0.00 -> 35.2 mm, vias 0 -> 2
- net TVCZ: track 0.00 -> 35.0 mm, vias 0 -> 1
- net SWCLK: track 0.00 -> 35.0 mm, vias 0 -> 2
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